File: EDA-kicad/audio.kicad_sch (KiCad schematic)
At the start: 8 parts, among them J4 SJ2-35894B-SMT-TR, U3 CODEC-TLV320AIC3204IRHBR

Commit message: Finished audio schematic
Parts:
- removed LS1, LS2: CMR-15062S-67, SPIRIT-footprints:SPEAKER_CMR-15062S-67, symbol SPIRIT-components:CMR-15062S-67
- added C26, C28: 10uF, symbol Device:C
- added C27: 20uF, symbol Device:C
- added C29, C50, C52, C53, C59, C62: 1uF, symbol Device:C
- added C48, C49, C51, C56, C57, C60, C63, C64, C65: 0.1uF, symbol Device:C
- added C54, C55: 47uF, symbol Device:C
- added C58, C61: 4.7nF, symbol Device:C
- added LS3, LS4: AS01506MS-SC15-WP-2-R, SPIRIT-footprints:AS01506MS-SC15-WP-2-R, symbol SPIRIT-components:AS01506MS-SC15-WP-2-R
- added R38: 2.7KΩ, symbol Device:R
- added R39, R40: 1KΩ, symbol Device:R
- added U12, U5: IM68A130A, SPIRIT-footprints:SMD-PG-TLGA-4-2-V, symbol SPIRIT-components:IM68A130A
- added U13, U14: TPA2038D1YFFR, SPIRIT-footprints:TPA2038D1YFFR, symbol SPIRIT-components:TPA2038D1YFFR
Connections:
- net AUDIO_MIC_DATA: now also U3.5 (DOUT/MFP2); no longer MK1.6 (DATA_OUT), R3.2
- net GND: now also J4.1, U3.12 (SPI_SELECT), U3.33 (EP), C26.2, C27.1, C28.1, C29.1, C48.1, C49.1, C51.1, C57.2, C58.2, C59.1, C60.1, C61.2, C62.1, C64.2, C65.1, U12.2 (GND), U12.4 (GND), U13.A2 (GAIN), U13.B3 (PGND), U14.A2 (GAIN), U14.B3 (PGND), U5.2 (GND), U5.4 (GND)
- net MIC-SWITCH: now also C49.2, C51.2, U12.3 (VDD), U5.3 (VDD)
- net VCC: no longer U3.24 (AVDD)
- net JACK_AUDIO_RIGHT: now reaches J4.2
- net JACK_AUDIO_RIGHT: now also C55.1
- net JACK_AUDIO_LEFT: now reaches J4.3
- net JACK_AUDIO_LEFT: now also C54.1
- net JACK_MIC: now reaches J4.4
- net JACK_MIC: now also U3.8 (SCLK/MFP3), C53.2, R38.2
- net at U3.13 (IN1_L): now also C50.1
- net at U3.14 (IN1_R): now also C52.1
- net at U3.18 (REF): now also C26.1
- net at U3.19 (MICBIAS): now also R38.1
- net at U3.21 (IN3_R): now also C53.1
- net AMP_AUDIO_LEFT: now reaches U3.22 (LOL)
- net AMP_AUDIO_LEFT: now also R39.1
- net AMP_AUDIO_RIGHT: now reaches U3.23 (LOR)
- net AMP_AUDIO_RIGHT: now also R40.1
- net at U3.25 (HPL): now also C54.2
- net 3V3B: now reaches U3.26 (LDOIN/HPVDD)
- net 3V3B: now also U3.30 (LDO_SELECT), U3.6 (IOVDD), C28.2, C29.2, C48.2
- net at U3.27 (HPR): now also C55.2
- net 1V8: now reaches U3.29 (DVDD)
- net 1V8: now also U3.24 (AVDD), C27.2
- net AUDIO_RESET: now reaches U3.31 (~{RESET})
- net AUDIO_SOUND_DATA: now reaches U3.4 (DIN/MFP1)
- new net: LS3.N, U13.A3 (VO-)
- new net: LS3.P, U13.C3 (VO+)
- new net: C63.1, U14.C1 (IN-)
- new net: C61.1, C63.2, R40.2
- new net: C57.1, U13.A1 (IN+)
- new net: LS4.N, U14.A3 (VO-)
- new net: LS4.P, U14.C3 (VO+)
- new net: C50.2, U5.1 (OUT)
- new net: C64.1, U14.A1 (IN+)
- new net: C56.1, U13.C1 (IN-)
- new net: C56.2, C58.1, R39.2
- new net: MK1.6 (DATA_OUT), R3.2
- new net: C52.2, U12.1 (OUT)
- new net SYS: C59.2, C60.2, C62.2, C65.2, U13.B1 (VDD), U13.B2 (PVDD), U13.C2 (EN), U14.B1 (VDD), U14.B2 (PVDD), U14.C2 (EN)
- no-connect marks 2 -> 3
Other:
- note added: "Add ferrite bead in series with avdd input before dvdd input to reduce ripple if necesary -Engi"
- note added: "Audio amplifiers & speakers"
- note added: "CODEC & microphones"
- note added: "Enable is tied to SYS for now. Can be hooked up to CM5 GPIO to allow for audio disable and save a bit of power. -Engi"
- note added: "Headphone Jack"
- note added: "Jack pinout wired to use CTIA standard -Engi"
- note added: "Left MIC"
- note added: "Place DC-Blocking caps as close to the CODEC as possible -Engi"
- note added: "Place lowest values closest to IC -Engi"
- note added: "Right MIC"
- moved on the sheet: C5, C6, J4, MK1, R3, U3
